File: MCU_v2.sch (EAGLE design)
At the start: 29 parts, among them IC1 ATMEGA2560-16AU, Y1 CSTCE16M0V53-R0 16MHZ

Commit message: Board ready but still has some DRC errors
Parts:
- removed JP5: 10x1F-H8.5, SmartPrj:PINHD-1X10_ARD
- removed JP6: 8x1F-H8.5, SmartPrj:PINHD-1X8
- added GPS_INT: 8x1F-H8.5, pinhead:PINHD-1X4
- added JP_BT: (no value), pinhead:PINHD-1X2
- D1: value CD1206-S01575 -> (none)
- renumbered JP1 to DIGITAL, JP2 to POWER, JP3 to SD, JP4 to GPS, JP7 to PWM, JP8 to LCD, JP9 to ICSP, LED1 to ON, LED2 to LED_13, S1 to RESET, Y1 to XTAL
Connections:
- removed net N$4: IC1.(OC0A/OC1C/PCINT7)PB7, JP5.5, R5.1
- removed net PB4: IC1.(OC2A/PCINT4)PB4, JP5.8
- removed net PB5: IC1.(OC1A/PCINT5)PB5, JP5.7
- new net PB7: IC1.(OC0A/OC1C/PCINT7)PB7, JP_BT.1, R4.2, R5.1
- net AREF: no longer JP5.3
- net GND: no longer JP5.4
- net PB6: now also JP_BT.2; no longer JP5.6, R4.2
- net PH5: no longer JP5.10
- net PH6: no longer JP5.9
- net RXD1: now also GPS_INT.3; no longer JP6.3
- net RXD2: no longer JP6.5
- net RXD3: no longer JP6.7
- net SCL: now also GPS_INT.1; no longer JP5.1, JP6.1
- net SDA: now also GPS_INT.2; no longer JP5.2, JP6.2
- net TXD1: now also GPS_INT.4; no longer JP6.4
- net TXD2: no longer JP6.6
- net TXD3: no longer JP6.8
Other:
- note removed: "10"
- note removed: "11"
- note removed: "14"
- note removed: "15"
- note removed: "16"
- note removed: "17"
- note removed: "18"
- note removed: "19"
- note removed: "8"
- note removed: "9"
